File: pcb/60x60_monochrome/LED_matrix.sch (KiCad schematic (older format))
At the start: 11 parts, among them U3 NPIC6C595, U4 M54564FP

Commit message: - add pins to the sheets, add reset/boot circuit
Changed lines of the file:
@@
 	3400 2350 3750 2350
 $Comp
-L GND #PWR25
+L GND #PWR027
 U 1 1 5BD6DD18
 P 3250 4950
-F 0 "#PWR25" H 3250 4700 50  0001 C CNN
+F 0 "#PWR027" H 3250 4700 50  0001 C CNN
 F 1 "GND" H 3250 4800 50  0000 C CNN
 F 2 "" H 3250 4950 50  0001 C CNN
@@
 $EndComp
 $Comp
-L GND #PWR22
+L GND #PWR028
 U 1 1 5BD6DD1E
 P 2650 4700
-F 0 "#PWR22" H 2650 4450 50  0001 C CNN
+F 0 "#PWR028" H 2650 4450 50  0001 C CNN
 F 1 "GND" H 2650 4550 50  0000 C CNN
 F 2 "" H 2650 4700 50  0001 C CNN
@@
 CAT_DATA
 $Comp
-L +3.3V #PWR23
+L +3.3V #PWR029
 U 1 1 5BD6DD38
 P 2700 4400
-F 0 "#PWR23" H 2700 4250 50  0001 C CNN
+F 0 "#PWR029" H 2700 4250 50  0001 C CNN
 F 1 "+3.3V" H 2700 4540 50  0000 C CNN
 F 2 "" H 2700 4400 50  0001 C CNN
@@
 $EndComp
 $Comp
-L +5V #PWR24
+L +5V #PWR030
 U 1 1 5BD6DD46
 P 3250 3450
-F 0 "#PWR24" H 3250 3300 50  0001 C CNN
+F 0 "#PWR030" H 3250 3300 50  0001 C CNN
 F 1 "+5V" H 3250 3590 50  0000 C CNN
 F 2 "" H 3250 3450 50  0001 C CNN
@@
 C1
 $Comp
-L GND #PWR27
+L GND #PWR031
 U 1 1 5BD6E38D
 P 6750 4600
-F 0 "#PWR27" H 6750 4350 50  0001 C CNN
+F 0 "#PWR031" H 6750 4350 50  0001 C CNN
 F 1 "GND" H 6750 4450 50  0000 C CNN
 F 2 "" H 6750 4600 50  0001 C CNN
@@
 NoConn ~ 7200 3500
 $Comp
-L +5V #PWR26
+L +5V #PWR032
 U 1 1 5BD6E3A7
 P 6750 3200
-F 0 "#PWR26" H 6750 3050 50  0001 C CNN
+F 0 "#PWR032" H 6750 3050 50  0001 C CNN
 F 1 "+5V" H 6750 3340 50  0000 C CNN
 F 2 "" H 6750 3200 50  0001 C CNN
@@
 	1    0    0    -1
 $EndComp
+Text HLabel 5900 3600 0    60   Input ~ 0
+LEDS_A0
+Text HLabel 5900 3700 0    60   Input ~ 0
+LEDS_A1
+Text HLabel 5900 3800 0    60   Input ~ 0
+LEDS_A2
+Text HLabel 5900 3900 0    60   Input ~ 0
+LEDS_A3
+Text HLabel 5900 4000 0    60   Input ~ 0
+LEDS_A4
+Text HLabel 5900 4100 0    60   Input ~ 0
+LEDS_A5
+Text HLabel 5900 4200 0    60   Input ~ 0
+LEDS_A6
+Text HLabel 5900 4300 0    60   Input ~ 0
+LEDS_A7
+Text HLabel 2250 3850 0    60   Input ~ 0
+CAT_CLK
+Text HLabel 2250 3750 0    60   Input ~ 0
+CAT_DATA
+Text HLabel 2250 4050 0    60   Input ~ 0
+CAT_STROBE
 $EndSCHEMATC
